Commit message: getting there

File: models/huron/huron.urdf (robot description, URDF)
Before this commit: robot huron, 16 links, 15 joints
Links:
- removed link l_ankle_roll_link
- removed link r_ankle_roll_link
- added link L_FOOT, mass 1.8533; visual mesh filename=meshes/stl_meshes/l_ankle_roll_link.STL scale=1 1 1
- added link R_FOOT, mass 1.8533; visual mesh filename=meshes/stl_meshes/r_ankle_roll_link.STL scale=1 1 1
- added link dummy, mass 0.000863223621815312
- link base_footprint: geometry visual mesh filename=meshes/stl_meshes/base_link.STL scale=1 1 1
- link l_ankle_pitch_link: geometry visual mesh filename=meshes/stl_meshes/l_ankle_pitch_link.STL scale=1 1 1
- link l_hip_pitch_link: geometry visual mesh filename=meshes/stl_meshes/l_hip_pitch_link.STL scale=1 1 1
- link l_hip_roll_link: geometry visual mesh filename=meshes/stl_meshes/l_hip_roll_link.STL scale=1 1 1
- link l_hip_yaw_link: geometry visual mesh filename=meshes/stl_meshes/l_hip_yaw_link.STL scale=1 1 1
- link l_knee_pitch_link: geometry visual mesh filename=meshes/stl_meshes/l_knee_pitch_link.STL scale=1 1 1
- link r_ankle_pitch_link: geometry visual mesh filename=meshes/stl_meshes/r_ankle_pitch_link.STL scale=1 1 1
- link r_hip_pitch_link: geometry visual mesh filename=meshes/stl_meshes/r_hip_pitch_link.STL scale=1 1 1
- link r_hip_roll_link: geometry visual mesh filename=meshes/stl_meshes/r_hip_roll_link.STL scale=1 1 1
- link r_hip_yaw_link: geometry visual mesh filename=meshes/stl_meshes/r_hip_yaw_link.STL scale=1 1 1
- link r_knee_pitch_link: geometry visual mesh filename=meshes/stl_meshes/r_knee_pitch_link.STL scale=1 1 1
Joints:
- added joint dummy_fixed: type fixed, parent dummy, child base_footprint, origin xyz=0 0 0 rpy=0 0 -1.57079633
- joint base_fixed: child base_footprint -> dummy
- joint l_ankle_pitch_joint: limit lower=-0.5236 upper=0.1745 effort=1000 velocity=3 -> lower=-3.1416 upper=3.1416 effort=1000 velocity=40; type revolute -> continuous
- joint l_ankle_roll_joint: child l_ankle_roll_link -> L_FOOT; limit lower=-0.3491 upper=0.3491 effort=1000 velocity=3 -> lower=-3.1416 upper=3.1416 effort=1000 velocity=40; type revolute -> continuous
- joint l_hip_pitch_joint: limit lower=-1.2217 upper=1.2217 effort=1000 velocity=3 -> lower=-3.1416 upper=3.1416 effort=1000 velocity=40; type revolute -> continuous
- joint l_hip_roll_joint: limit lower=-0.01 upper=0.5236 effort=1000 velocity=3 -> lower=-3.1416 upper=3.1416 effort=1000 velocity=40; type revolute -> continuous
- joint l_hip_yaw_joint: limit lower=-3.1416 upper=3.1416 effort=1000 velocity=3 -> lower=-3.1416 upper=3.1416 effort=1000 velocity=40; type revolute -> continuous
- joint l_knee_pitch_joint: limit lower=-1.570796327 upper=1.570796327 effort=1000 velocity=3 -> lower=-3.1416 upper=3.1416 effort=1000 velocity=40; type revolute -> continuous
- joint r_ankle_pitch_joint: limit lower=-0.5236 upper=0.1745 effort=1000 velocity=3 -> lower=-3.1416 upper=3.1416 effort=1000 velocity=40; type revolute -> continuous
- joint r_ankle_roll_joint: child r_ankle_roll_link -> R_FOOT; limit lower=-0.3491 upper=0.3491 effort=1000 velocity=3 -> lower=-3.1416 upper=3.1416 effort=1000 velocity=40; type revolute -> continuous
- joint r_hip_pitch_joint: limit lower=-1.2217 upper=1.2217 effort=1000 velocity=3 -> lower=-3.1416 upper=3.1416 effort=1000 velocity=40; type revolute -> continuous
- joint r_hip_roll_joint: limit lower=-0.5236 upper=0.01 effort=1000 velocity=3 -> lower=-3.1416 upper=3.1416 effort=1000 velocity=40; type revolute -> continuous
- joint r_hip_yaw_joint: limit lower=-3.1416 upper=3.1416 effort=1000 velocity=3 -> lower=-3.1416 upper=3.1416 effort=1000 velocity=40; type revolute -> continuous
- joint r_knee_pitch_joint: limit lower=-1.570796327 upper=1.570796327 effort=1000 velocity=3 -> lower=-3.1416 upper=3.1416 effort=1000 velocity=40; type revolute -> continuous
